Commit message: manipulator

File: resource/description/manipulator.urdf.xacro (robot description, xacro)
@@ -4,11 +4,11 @@
   <link name="world" />
   <!-- Include arm and hand xacro files-->
-  <xacro:include filename="$(find manipulator)/description/panda_arm.xacro" />
-  <xacro:include filename="$(find manipulator)/description/panda_hand.xacro" />
+  <xacro:include filename="panda_arm.xacro" />
+  <xacro:include filename="panda_hand.xacro" />
   <!-- call the arm macro-->
   <xacro:panda_arm />
   <!-- call the hand macro-->
   <xacro:panda_hand ns="panda" rpy="0 0 ${-pi/4}" connected_to="panda_link8" />
-  <xacro:include filename="$(find manipulator)/description/manipulator.gazebo.xacro" />
-  <xacro:include filename="$(find manipulator)/description/manipulator.control.xacro" />
+  <xacro:include filename="manipulator.gazebo.xacro" />
+  <xacro:include filename="manipulator.control.xacro" />
 </robot>

File: resource/description/panda_arm.xacro (robot description, xacro)
@@ -42,5 +42,5 @@
       <parent link="world" />
       <child link="${arm_id}_link0" />
-      <origin xyz="0.0 0.0 0.0" rpy="0.0 0.0 0.0" />
+      <origin xyz="0.0 0.0 1.0" rpy="0.0 0.0 0.0" />
       <dynamics damping="${joint_damping}" />
     </joint>
@@ -48,10 +48,10 @@
       <visual>
         <geometry>
-          <mesh filename="file://$(find manipulator)/meshes/visual/link0.dae" />
-        </geometry>
-      </visual>
-      <collision>
-        <geometry>
-          <mesh filename="file://$(find manipulator)/meshes/collision/link0.stl" />
+          <mesh filename="file://$(find manipulator)/resource/meshes/visual/link0.dae" />
+        </geometry>
+      </visual>
+      <collision>
+        <geometry>
+          <mesh filename="file://$(find manipulator)/resource/meshes/collision/link0.stl" />
         </geometry>
       </collision>
@@ -65,10 +65,10 @@
       <visual>
         <geometry>
-          <mesh filename="file://$(find manipulator)/meshes/visual/link1.dae" />
-        </geometry>
-      </visual>
-      <collision>
-        <geometry>
-          <mesh filename="file://$(find manipulator)/meshes/collision/link1.stl" />
+          <mesh filename="file://$(find manipulator)/resource/meshes/visual/link1.dae" />
+        </geometry>
+      </visual>
+      <collision>
+        <geometry>
+          <mesh filename="file://$(find manipulator)/resource/meshes/collision/link1.stl" />
         </geometry>
       </collision>
@@ -94,10 +94,10 @@
       <visual>
         <geometry>
-          <mesh filename="file://$(find manipulator)/meshes/visual/link2.dae" />
-        </geometry>
-      </visual>
-      <collision>
-        <geometry>
-          <mesh filename="file://$(find manipulator)/meshes/collision/link2.stl" />
+          <mesh filename="file://$(find manipulator)/resource/meshes/visual/link2.dae" />
+        </geometry>
+      </visual>
+      <collision>
+        <geometry>
+          <mesh filename="file://$(find manipulator)/resource/meshes/collision/link2.stl" />
         </geometry>
       </collision>
@@ -123,10 +123,10 @@
       <visual>
         <geometry>
-          <mesh filename="file://$(find manipulator)/meshes/visual/link3.dae" />
-        </geometry>
-      </visual>
-      <collision>
-        <geometry>
-          <mesh filename="file://$(find manipulator)/meshes/collision/link3.stl" />
+          <mesh filename="file://$(find manipulator)/resource/meshes/visual/link3.dae" />
+        </geometry>
+      </visual>
+      <collision>
+        <geometry>
+          <mesh filename="file://$(find manipulator)/resource/meshes/collision/link3.stl" />
         </geometry>
       </collision>
@@ -153,10 +153,10 @@
       <visual>
         <geometry>
-          <mesh filename="file://$(find manipulator)/meshes/visual/link4.dae" />
-        </geometry>
-      </visual>
-      <collision>
-        <geometry>
-          <mesh filename="file://$(find manipulator)/meshes/collision/link4.stl" />
+          <mesh filename="file://$(find manipulator)/resource/meshes/visual/link4.dae" />
+        </geometry>
+      </visual>
+      <collision>
+        <geometry>
+          <mesh filename="file://$(find manipulator)/resource/meshes/collision/link4.stl" />
         </geometry>
       </collision>
@@ -183,10 +183,10 @@
       <visual>
         <geometry>
-          <mesh filename="file://$(find manipulator)/meshes/visual/link5.dae" />
-        </geometry>
-      </visual>
-      <collision>
-        <geometry>
-          <mesh filename="file://$(find manipulator)/meshes/collision/link5.stl" />
+          <mesh filename="file://$(find manipulator)/resource/meshes/visual/link5.dae" />
+        </geometry>
+      </visual>
+      <collision>
+        <geometry>
+          <mesh filename="file://$(find manipulator)/resource/meshes/collision/link5.stl" />
         </geometry>
       </collision>
@@ -212,10 +212,10 @@
       <visual>
         <geometry>
-          <mesh filename="file://$(find manipulator)/meshes/visual/link6.dae" />
-        </geometry>
-      </visual>
-      <collision>
-        <geometry>
-          <mesh filename="file://$(find manipulator)/meshes/collision/link6.stl" />
+          <mesh filename="file://$(find manipulator)/resource/meshes/visual/link6.dae" />
+        </geometry>
+      </visual>
+      <collision>
+        <geometry>
+          <mesh filename="file://$(find manipulator)/resource/meshes/collision/link6.stl" />
         </geometry>
       </collision>
@@ -241,10 +241,10 @@
       <visual>
         <geometry>
-          <mesh filename="file://$(find manipulator)/meshes/visual/link7.dae" />
-        </geometry>
-      </visual>
-      <collision>
-        <geometry>
-          <mesh filename="file://$(find manipulator)/meshes/collision/link7.stl" />
+          <mesh filename="file://$(find manipulator)/resource/meshes/visual/link7.dae" />
+        </geometry>
+      </visual>
+      <collision>
+        <geometry>
+          <mesh filename="file://$(find manipulator)/resource/meshes/collision/link7.stl" />
         </geometry>
       </collision>

File: resource/description/panda_hand.xacro (robot description, xacro)
@@ -12,10 +12,10 @@
             <visual>
                 <geometry>
-                    <mesh filename="file://$(find manipulator)/meshes/visual/hand.dae" />
+                    <mesh filename="file://$(find manipulator)/resource/meshes/visual/hand.dae" />
                 </geometry>
             </visual>
             <collision>
                 <geometry>
-                    <mesh filename="file://$(find manipulator)/meshes/collision/hand.stl" />
+                    <mesh filename="file://$(find manipulator)/resource/meshes/collision/hand.stl" />
                 </geometry>
             </collision>
