Commit message: update

File: resources/robot_description/manipulator.control.xacro (robot description, xacro)
@@ -3,74 +3,6 @@
     <gazebo>
         <plugin filename="libgazebo_ros2_control.so" name="gazebo_ros2_control">
-            <parameters>$(find manipulator)/resources/controllers/controllers.yaml</parameters>
+            <parameters>$(find manipulator)/config/controllers.yaml</parameters>
         </plugin>
     </gazebo>
-    <ros2_control name="GazeboSystem" type="system">
-        <hardware>
-            <plugin>gazebo_ros2_control/GazeboSystem</plugin>
-        </hardware>
-        <joint name="panda_joint1">
-            <command_interface name="position">
-                <!-- <param name="min">-2.8973</param> -->
-                <!-- <param name="max">2.8973</param> -->
-            </command_interface>
-            <state_interface name="position" />
-            <state_interface name="velocity" />
-            <state_interface name="effort" />
-        </joint>
-        <joint name="panda_joint2">
-            <command_interface name="position">
-                <!-- <param name="min">-1.7628</param> -->
-                <!-- <param name="max">1.7628</param> -->
-            </command_interface>
-            <state_interface name="position" />
-            <state_interface name="velocity" />
-            <state_interface name="effort" />
-        </joint>
-        <joint name="panda_joint3">
-            <command_interface name="position">
-                <!-- <param name="min">-2.8973</param> -->
-                <!-- <param name="max">2.8973</param> -->
-            </command_interface>
-            <state_interface name="position" />
-            <state_interface name="velocity" />
-            <state_interface name="effort" />
-        </joint>
-        <joint name="panda_joint4">
-            <command_interface name="position">
-                <!-- <param name="min">-3.0718</param> -->
-                <!-- <param name="max">-0.0698</param> -->
-            </command_interface>
-            <state_interface name="position" />
-            <state_interface name="velocity" />
-            <state_interface name="effort" />
-        </joint>
-        <joint name="panda_joint5">
-            <command_interface name="position">
-                <!-- <param name="min">-2.8973</param> -->
-                <!-- <param name="max">2.8973</param> -->
-            </command_interface>
-            <state_interface name="position" />
-            <state_interface name="velocity" />
-            <state_interface name="effort" />
-        </joint>
-        <joint name="panda_joint6">
-            <command_interface name="position">
-                <!-- <param name="min">-0.0175</param> -->
-                <!-- <param name="max">3.7525</param> -->
-            </command_interface>
-            <state_interface name="position" />
-            <state_interface name="velocity" />
-            <state_interface name="effort" />
-        </joint>
-        <joint name="panda_joint7">
-            <command_interface name="position">
-                <!-- <param name="min">-0.0175</param> -->
-                <!-- <param name="max">3.7525</param> -->
-            </command_interface>
-            <state_interface name="position" />
-            <state_interface name="velocity" />
-            <state_interface name="effort" />
-        </joint>
-    </ros2_control>
 </robot>

File: resources/robot_description/manipulator.urdf (robot description, URDF)
Before this commit: robot panda, 12 links, 11 joints
Links:
- link panda_hand: geometry collision mesh filename=file:///home/luisc/ws_manipulator/install/manipulator/share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; visual mesh filename=file:///home/luisc/ws_manipulator/install/manipulator/share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
- link panda_link0: geometry collision mesh filename=file:///home/luisc/ws_manipulator/install/manipulator/share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; visual mesh filename=file:///home/luisc/ws_manipulator/install/manipulator/share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
- link panda_link1: geometry collision mesh filename=file:///home/luisc/ws_manipulator/install/manipulator/share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; visual mesh filename=file:///home/luisc/ws_manipulator/install/manipulator/share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
- link panda_link2: geometry collision mesh filename=file:///home/luisc/ws_manipulator/install/manipulator/share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; visual mesh filename=file:///home/luisc/ws_manipulator/install/manipulator/share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
- link panda_link3: geometry collision mesh filename=file:///home/luisc/ws_manipulator/install/manipulator/share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; visual mesh filename=file:///home/luisc/ws_manipulator/install/manipulator/share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
- link panda_link4: geometry collision mesh filename=file:///home/luisc/ws_manipulator/install/manipulator/share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; visual mesh filename=file:///home/luisc/ws_manipulator/install/manipulator/share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
- link panda_link5: geometry collision mesh filename=file:///home/luisc/ws_manipulator/install/manipulator/share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; visual mesh filename=file:///home/luisc/ws_manipulator/install/manipulator/share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
- link panda_link6: geometry collision mesh filename=file:///home/luisc/ws_manipulator/install/manipulator/share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; visual mesh filename=file:///home/luisc/ws_manipulator/install/manipulator/share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
- link panda_link7: geometry collision mesh filename=file:///home/luisc/ws_manipulator/install/manipulator/share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; visual mesh filename=file:///home/luisc/ws_manipulator/install/manipulator/share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
Joints:
- joint robot_to_world: origin xyz=0.0 0.0 0.0 rpy=0.0 0.0 0.0 -> xyz=0.0 0.0 1.0 rpy=0.0 0.0 0.0

File: resources/robot_description/panda_ros2_control.xacro (robot description, xacro)
@@ -8,4 +8,5 @@
       <joint name="${prefix}panda_joint1">
         <command_interface name="position"/>
+        <command_interface name="effort"/>
         <state_interface name="position"/>
         <state_interface name="velocity"/>
@@ -14,4 +15,5 @@
       <joint name="${prefix}panda_joint2">
         <command_interface name="position"/>
+        <command_interface name="effort"/>
         <state_interface name="position"/>
         <state_interface name="velocity"/>
@@ -20,4 +22,5 @@
       <joint name="${prefix}panda_joint3">
         <command_interface name="position"/>
+        <command_interface name="effort"/>
         <state_interface name="position"/>
         <state_interface name="velocity"/>
@@ -26,4 +29,5 @@
       <joint name="${prefix}panda_joint4">
         <command_interface name="position"/>
+        <command_interface name="effort"/>
         <state_interface name="position"/>
         <state_interface name="velocity"/>
@@ -32,4 +36,5 @@
       <joint name="${prefix}panda_joint5">
         <command_interface name="position"/>
+        <command_interface name="effort"/>
         <state_interface name="position"/>
         <state_interface name="velocity"/>
@@ -38,4 +43,5 @@
       <joint name="${prefix}panda_joint6">
         <command_interface name="position"/>
+        <command_interface name="effort"/>
         <state_interface name="position"/>
         <state_interface name="velocity"/>
@@ -44,4 +50,5 @@
       <joint name="${prefix}panda_joint7">
         <command_interface name="position"/>
+        <command_interface name="effort"/>
         <state_interface name="position"/>
         <state_interface name="velocity"/>
